File: nRF_beacon/AUDIO.kicad_sch (KiCad schematic)
At the start: 10 parts, among them U1 nRF54L15, U2 MAX98357A

Commit message: Finished typical application nRF. Added audio-block in root sheet.
Parts:
- removed LS1: AS07104PO-R, symbol Device:Speaker
- removed R2: 1M, symbol Device:R_Small
- removed U1: nRF54L15, Ekse:QFN48_6X6_NOR, symbol Ekse:nRF54L15
Connections:
- net OUTN: now reaches C8.1, L3.2
- net OUTP: now reaches C9.1, L2.2
- net ~{SD_MODE}: now reaches U2.4 (~{SD_MODE})
Other:
- note removed: "Mode: (Left/2 + Right/2)"

Commit message: Added MPN and footprints for all components on nRF general application
Parts:
- removed L2, L3: Ferrite, symbol Device:L_Ferrite_Small
- added FB2, FB3: FerriteBead_Small, symbol Device:FerriteBead_Small
- renumbered C10 to C17, C11 to C18, C8 to C19, C9 to C20, U2 to U3
Connections:
- net OUTN: now also FB3.2
- net OUTP: now also FB2.2
- net at U3.10 (OUTN): now also FB3.1
- net at U3.9 (OUTP): now also FB2.1

Commit message: Added buck configuration for AUDIO 3.3V power. Removed USB input
Connections:
- net +5V renamed VDD_AUDIO
Other:
- note added: "3.3V"
- note added: "From nPM1300"
Changed lines of the file:
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@@
+		)
+	)
+	(text "From nPM1300"
+		(exclude_from_sim no)
+		(at 173.736 68.834 0)
+		(effects
+			(font
+				(size 1.27 1.27)
+			)
 		)
 	)
@@
 			(font
 				(size 3.81 3.81)
+			)
+		)
+	)
+	(text "3.3V"
+		(exclude_from_sim no)
+		(at 172.72 66.548 0)
+		(effects
+			(font
+				(size 1.27 1.27)
 			)
 		)
@@
 	)
 	(symbol
+		(lib_id "power:+3V3")
+		(at 172.72 74.93 0)
+		(unit 1)
+		(exclude_from_sim no)
+		(in_bom yes)
+		(on_board yes)
+		(dnp no)
+		(property "Reference" "#PWR028"
+			(at 172.72 78.74 0)
+			(effects
+				(font
+					(size 1.27 1.27)
+				)
+				(hide yes)
+			)
+		)
+		(property "Value" "VDD_AUDIO"
+			(at 172.72 71.374 0)
+			(effects
+				(font
+					(size 1.27 1.27)
+				)
+			)
+		)
+		(property "Footprint" ""
+			(at 172.72 74.93 0)
+			(effects
+				(font
+					(size 1.27 1.27)
+				)
+				(hide yes)
+			)
+		)
+		(property "Datasheet" ""
+			(at 172.72 74.93 0)
+			(effects
+				(font
+					(size 1.27 1.27)
+				)
+				(hide yes)
+			)
+		)
+		(property "Description" "Power symbol creates a global label with name \"+3V3\""
+			(at 172.72 74.93 0)
+			(effects
+				(font
+					(size 1.27 1.27)
+				)
+				(hide yes)
+			)
+		)
+		(pin "1"
+		)
+		(instances
+			(project ""
+				(path "/1290e5f5-b91f-4d6e-b440-6b78e8fdc212/437e71df-bd9b-467f-b101-39f98a623051"
+					(reference "#PWR028")
+					(unit 1)
+				)
+			)
+		)
+	)
+	(symbol
 		(lib_id "Ekse:MAX98357A")
 		(at 140.97 93.98 0)
@@
 					(unit 1)
 				)
-			)
-		)
-	)
-	(symbol
-		(lib_id "power:+5V")
-		(at 172.72 74.93 0)
-		(unit 1)
-		(exclude_from_sim no)
-		(in_bom yes)
-		(on_board yes)
-		(dnp no)
-		(fields_autoplaced yes)
-		(property "Reference" "#PWR024"
-			(at 172.72 78.74 0)
-			(effects
-				(font
-					(size 1.27 1.27)
-				)
-				(hide yes)
-			)
-		)
-		(property "Value" "+5V"
-			(at 172.72 69.85 0)
-			(effects
-				(font
-					(size 1.27 1.27)
-				)
-			)
-		)
-		(property "Footprint" ""
-			(at 172.72 74.93 0)
-			(effects
-				(font
-					(size 1.27 1.27)
-				)
-				(hide yes)
-			)
-		)
-		(property "Datasheet" ""
-			(at 172.72 74.93 0)
-			(effects
-				(font
-					(size 1.27 1.27)
-				)
-				(hide yes)
-			)
-		)
-		(property "Description" "Power symbol creates a global label with name \"+5V\""
-			(at 172.72 74.93 0)
-			(effects
-				(font
-					(size 1.27 1.27)
-				)
-				(hide yes)
-			)
-		)
-		(pin "1"
-		)
-		(instances
-			(project "nRF_beacon"
-				(path "/1290e5f5-b91f-4d6e-b440-6b78e8fdc212/437e71df-bd9b-467f-b101-39f98a623051"
-					(reference "#PWR024")
-					(unit 1)
-				)

Commit message: Updated nPM schematic. Added TWI and debug connector
Parts:
- added R1: 1M, symbol Device:R_Small
Connections:
- net VDD_AUDIO: now also R1.1
- net ~{SD_MODE}: no longer names the net of U3.4 (~{SD_MODE})
- net ~{SD_MODE}: now also R1.2
Other:
- note added: "Mode: (Left/2 + Right/2)"
Changed lines of the file:
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@@
+		)
+	)
+	(text "Mode: \n(Left/2 + Right/2)"
+		(exclude_from_sim no)
+		(at 113.284 99.314 0)
+		(effects
+			(font
+				(size 0.635 0.635)
+			)
 		)
 	)
@@
 	(wire
 		(pts
-			(xy 109.22 96.52) (xy 125.73 96.52)
-		)
-		(stroke
-			(width 0)
-			(type default)
-		)
-	)
-	(wire
-		(pts
 			(xy 172.72 78.74) (xy 172.72 81.28)
 		)
@@
 	(wire
 		(pts
+			(xy 115.57 93.98) (xy 115.57 96.52)
+		)
+		(stroke
+			(width 0)
+			(type default)
+		)
+	)
+	(wire
+		(pts
 			(xy 158.75 78.74) (xy 158.75 81.28)
 		)
@@
 	(wire
 		(pts
+			(xy 118.11 96.52) (xy 115.57 96.52)
+		)
+		(stroke
+			(width 0)
+			(type default)
+		)
+	)
+	(wire
+		(pts
 			(xy 124.46 111.76) (xy 124.46 113.03)
 		)
@@
 		(pts
 			(xy 109.22 81.28) (xy 125.73 81.28)
+		)
+		(stroke
+			(width 0)
+			(type default)
+		)
+	)
+	(wire
+		(pts
+			(xy 123.19 96.52) (xy 125.73 96.52)
 		)
 		(stroke
@@
 		)
 	)
-	(hierarchical_label "~{SD_MODE}"
-		(shape input)
-		(at 109.22 96.52 180)
-		(effects
-			(font
-				(size 1.27 1.27)
-			)
-			(justify right)
-		)
-	)
 	(hierarchical_label "DIN"
 		(shape input)
@@
 	(symbol
 		(lib_id "power:+3V3")
+		(at 115.57 93.98 0)
+		(unit 1)
+		(exclude_from_sim no)
+		(in_bom yes)
+		(on_board yes)
+		(dnp no)
+		(property "Reference" "#PWR024"
+			(at 115.57 97.79 0)
+			(effects
+				(font
+					(size 1.27 1.27)
+				)
+				(hide yes)
+			)
+		)
+		(property "Value" "VDD_AUDIO"
+			(at 115.57 90.424 0)
+			(effects
+				(font
+					(size 1.27 1.27)
+				)
+			)
+		)
+		(property "Footprint" ""
+			(at 115.57 93.98 0)
+			(effects
+				(font
+					(size 1.27 1.27)
+				)
+				(hide yes)
+			)
+		)
+		(property "Datasheet" ""
+			(at 115.57 93.98 0)
+			(effects
+				(font
+					(size 1.27 1.27)
+				)
+				(hide yes)
+			)
+		)
+		(property "Description" "Power symbol creates a global label with name \"+3V3\""
+			(at 115.57 93.98 0)
+			(effects
+				(font
+					(size 1.27 1.27)
+				)
+				(hide yes)
+			)
+		)
+		(pin "1"
+		)
+		(instances
+			(project "nRF_beacon"
+				(path "/1290e5f5-b91f-4d6e-b440-6b78e8fdc212/437e71df-bd9b-467f-b101-39f98a623051"
+					(reference "#PWR024")
+					(unit 1)
+				)
+			)
+		)
+	)
+	(symbol
+		(lib_id "power:+3V3")
 		(at 172.72 74.93 0)
 		(unit 1)
@@
 					(unit 1)
 				)
+			)
+		)
+	)
+	(symbol
+		(lib_id "Device:R_Small")
+		(at 120.65 96.52 90)
+		(unit 1)
+		(exclude_from_sim no)
+		(in_bom yes)
+		(on_board yes)
+		(dnp no)
+		(property "Reference" "R1"
+			(at 120.65 94.996 90)
+			(effects
+				(font
+					(size 1.016 1.016)
+				)
+			)
+		)
+		(property "Value" "1M"
+			(at 120.65 98.552 90)
+			(effects
+				(font
+					(size 1.27 1.27)
+				)
+			)
+		)
+		(property "Footprint" ""
+			(at 120.65 96.52 0)
+			(effects
+				(font
+					(size 1.27 1.27)
+				)
+				(hide yes)
+			)
+		)
+		(property "Datasheet" "~"
+			(at 120.65 96.52 0)
+			(effects
+				(font
+					(size 1.27 1.27)
+				)
+				(hide yes)
+			)
+		)
+		(property "Description" "Resistor, small symbol"
+			(at 120.65 96.52 0)
+			(effects
+				(font
+					(size 1.27 1.27)
+				)
+				(hide yes)
+			)
+		)
+		(pin "2"
+		)
+		(pin "1"
+		)
+		(instances
+			(project ""
+				(path "/1290e5f5-b91f-4d6e-b440-6b78e8fdc212/437e71df-bd9b-467f-b101-39f98a623051"
+					(reference "R1")
+					(unit 1)
+				)

Commit message: Finished first schematic draft. Ready for layout
Parts:
- C17: footprint (none) -> Capacitor_SMD:C_0603_1608Metric_Pad1.08x0.95mm_HandSolder; MPN (none) -> KGM15CR51E106KT; Price (none) -> 5.09
- C18: footprint (none) -> Capacitor_SMD:C_0201_0603Metric_Pad0.64x0.40mm_HandSolder; MPN (none) -> KGM03BR51E104KH; Price (none) -> 1.39
- C19, C20: footprint (none) -> Capacitor_SMD:C_0603_1608Metric_Pad1.08x0.95mm_HandSolder; MPN (none) -> C0603C221J5RACTM; Price (none) -> 1.3
- FB2, FB3: value FerriteBead_Small -> 1000; footprint (none) -> Capacitor_SMD:C_0805_2012Metric_Pad1.18x1.45mm_HandSolder; MPN (none) -> BLM21SP102SN1D; Price (none) -> 2.99
- R1: value 1M -> 634k; footprint (none) -> Resistor_SMD:R_0603_1608Metric_Pad0.98x0.95mm_HandSolder; MPN (none) -> CRCW0603634KDHTAP; Price (none) -> 3.89
- U3: MPN (none) -> MAX98357AETE+T; Price (none) -> 51.62
Changed lines of the file:
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@@
 			)
 		)
-		(property "Footprint" ""
+		(property "Footprint" "Capacitor_SMD:C_0603_1608Metric_Pad1.08x0.95mm_HandSolder"
 			(at 176.53 111.76 0)
 			(effects
@@
 			)
 		)
-		(property "MPN" ""
+		(property "MPN" "C0603C221J5RACTM"
 			(at 176.53 111.76 0)
 			(effects
@@
 			)
 		)
-		(property "Price" ""
+		(property "Price" "1.3"
 			(at 176.53 111.76 0)
 			(effects
@@
 			)
 		)
-		(property "Footprint" ""
+		(property "Footprint" "Capacitor_SMD:C_0201_0603Metric_Pad0.64x0.40mm_HandSolder"
 			(at 172.72 83.82 0)
 			(effects
@@
 			)
 		)
-		(property "MPN" ""
+		(property "MPN" "KGM03BR51E104KH"
 			(at 172.72 83.82 0)
 			(effects
@@
 			)
 		)
-		(property "Price" ""
+		(property "Price" "1.39"
 			(at 172.72 83.82 0)
 			(effects
@@
 			)
 		)
-		(property "Value" "FerriteBead_Small"
+		(property "Value" "1000"
 			(at 165.1 99.06 90)
 			(effects
@@
 			)
 		)
-		(property "Footprint" ""
+		(property "Footprint" "Capacitor_SMD:C_0805_2012Metric_Pad1.18x1.45mm_HandSolder"
 			(at 165.1 98.298 90)
 			(effects
@@
 			)
 		)
-		(property "MPN" ""
+		(property "MPN" "BLM21SP102SN1D"
 			(at 165.1 96.52 90)
 			(effects
@@
 			)
 		)
-		(property "Price" ""
+		(property "Price" "2.99"
 			(at 165.1 96.52 90)
 			(effects
@@
 			)
 		)
-		(property "Value" "FerriteBead_Small"
+		(property "Value" "1000"
 			(at 165.1 107.442 90)
 			(effects
@@
 			)
 		)
-		(property "Footprint" ""
+		(property "Footprint" "Capacitor_SMD:C_0805_2012Metric_Pad1.18x1.45mm_HandSolder"
 			(at 165.1 105.918 90)
 			(effects
@@
 			)
 		)
-		(property "MPN" ""
+		(property "MPN" "BLM21SP102SN1D"
 			(at 165.1 104.14 90)
 			(effects
@@
 			)
 		)
-		(property "Price" ""
+		(property "Price" "2.99"
 			(at 165.1 104.14 90)
 			(effects
@@
 			)
 		)
-		(property "MPN" ""
+		(property "MPN" "MAX98357AETE+T"
 			(at 140.97 93.98 0)
 			(effects
@@
 			)
 		)
-		(property "Price" ""
+		(property "Price" "51.62"
 			(at 140.97 93.98 0)
 			(effects
@@
 			)
 		)
-		(property "Value" "1M"
+		(property "Value" "634k"
 			(at 120.65 98.552 90)
 			(effects
@@
 			)
 		)
-		(property "Footprint" ""
+		(property "Footprint" "Resistor_SMD:R_0603_1608Metric_Pad0.98x0.95mm_HandSolder"
 			(at 120.65 96.52 0)
 			(effects
@@
 			)
 		)
+		(property "MPN" "CRCW0603634KDHTAP"
+			(at 120.65 96.52 90)
+			(effects
+				(font
+					(size 1.27 1.27)
+				)
+				(hide yes)
+			)
+		)
+		(property "Price" "3.89"
+			(at 120.65 96.52 90)
+			(effects
+				(font
+					(size 1.27 1.27)
+				)
+				(hide yes)
+			)
+		)
 		(pin "2"
 		)
@@
 			)
 		)
-		(property "Footprint" ""
+		(property "Footprint" "Capacitor_SMD:C_0603_1608Metric_Pad1.08x0.95mm_HandSolder"
 			(at 162.56 83.82 0)
 			(effects
@@
 			)
 		)
-		(property "MPN" ""
+		(property "MPN" "KGM15CR51E106KT"
 			(at 162.56 83.82 0)
 			(effects
@@
 			)
 		)
-		(property "Price" ""
+		(property "Price" "5.09"
 			(at 162.56 83.82 0)
 			(effects
@@
 			)
 		)
-		(property "Footprint" ""
+		(property "Footprint" "Capacitor_SMD:C_0603_1608Metric_Pad1.08x0.95mm_HandSolder"
 			(at 186.69 111.76 0)
 			(effects
@@
 			)
 		)
-		(property "MPN" ""
+		(property "MPN" "C0603C221J5RACTM"
 			(at 186.69 111.76 0)
 			(effects
@@
 			)
 		)
-		(property "Price" ""
+		(property "Price" "1.3"
 			(at 186.69 111.76 0)
 			(effects

Commit message: Began matching network layout
Parts:
- C17, C19, C20: footprint Capacitor_SMD:C_0603_1608Metric_Pad1.08x0.95mm_HandSolder -> Capacitor_SMD:C_0603_1608Metric
- C18: footprint Capacitor_SMD:C_0201_0603Metric_Pad0.64x0.40mm_HandSolder -> Capacitor_SMD:C_0201_0603Metric
- FB2, FB3: footprint Capacitor_SMD:C_0805_2012Metric_Pad1.18x1.45mm_HandSolder -> Capacitor_SMD:C_0805_2012Metric
- R1: footprint Resistor_SMD:R_0603_1608Metric_Pad0.98x0.95mm_HandSolder -> Resistor_SMD:R_0603_1608Metric
Changed lines of the file:
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@@
 			)
 		)
-		(property "Footprint" "Capacitor_SMD:C_0603_1608Metric_Pad1.08x0.95mm_HandSolder"
+		(property "Footprint" "Capacitor_SMD:C_0603_1608Metric"
 			(at 176.53 111.76 0)
 			(effects
@@
 			)
 		)
-		(property "Footprint" "Capacitor_SMD:C_0201_0603Metric_Pad0.64x0.40mm_HandSolder"
+		(property "Footprint" "Capacitor_SMD:C_0201_0603Metric"
 			(at 172.72 83.82 0)
 			(effects
@@
 			)
 		)
-		(property "Footprint" "Capacitor_SMD:C_0805_2012Metric_Pad1.18x1.45mm_HandSolder"
+		(property "Footprint" "Capacitor_SMD:C_0805_2012Metric"
 			(at 165.1 98.298 90)
 			(effects
@@
 			)
 		)
-		(property "Footprint" "Capacitor_SMD:C_0805_2012Metric_Pad1.18x1.45mm_HandSolder"
+		(property "Footprint" "Capacitor_SMD:C_0805_2012Metric"
 			(at 165.1 105.918 90)
 			(effects
@@
 			)
 		)
-		(property "Footprint" "Resistor_SMD:R_0603_1608Metric_Pad0.98x0.95mm_HandSolder"
+		(property "Footprint" "Resistor_SMD:R_0603_1608Metric"
 			(at 120.65 96.52 0)
 			(effects
@@
 			)
 		)
-		(property "Footprint" "Capacitor_SMD:C_0603_1608Metric_Pad1.08x0.95mm_HandSolder"
+		(property "Footprint" "Capacitor_SMD:C_0603_1608Metric"
 			(at 162.56 83.82 0)
 			(effects
@@
 			)
 		)
-		(property "Footprint" "Capacitor_SMD:C_0603_1608Metric_Pad1.08x0.95mm_HandSolder"
+		(property "Footprint" "Capacitor_SMD:C_0603_1608Metric"
 			(at 186.69 111.76 0)
 			(effects

Commit message: Added most of the components to nRF54 typical application layout
Connections:
- net Earth renamed GND
Changed lines of the file:
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@@
 			)
 		)
-		(property "Value" "Earth"
+		(property "Value" "GND"
 			(at 172.72 92.71 0)
 			(effects
@@
 			)
 		)
-		(property "Description" "Power symbol creates a global label with name \"Earth\""
+		(property "Description" "Power symbol creates a global label with name \"GND\""
 			(at 172.72 87.63 0)
 			(effects
@@
 			)
 		)
-		(property "Value" "Earth"
+		(property "Value" "GND"
 			(at 162.56 92.71 0)
 			(effects
@@
 			)
 		)
-		(property "Description" "Power symbol creates a global label with name \"Earth\""
+		(property "Description" "Power symbol creates a global label with name \"GND\""
 			(at 162.56 87.63 0)
 			(effects
@@
 			)
 		)
-		(property "Value" "Earth"
+		(property "Value" "GND"
 			(at 176.53 124.46 0)
 			(effects
@@
 			)
 		)
-		(property "Description" "Power symbol creates a global label with name \"Earth\""
+		(property "Description" "Power symbol creates a global label with name \"GND\""
 			(at 176.53 119.38 0)
 			(effects
@@
 			)
 		)
-		(property "Value" "Earth"
+		(property "Value" "GND"
 			(at 186.69 124.46 0)
 			(effects
@@
 			)
 		)
-		(property "Description" "Power symbol creates a global label with name \"Earth\""
+		(property "Description" "Power symbol creates a global label with name \"GND\""
 			(at 186.69 119.38 0)
 			(effects
@@
 			)
 		)
-		(property "Value" "Earth"
+		(property "Value" "GND"
 			(at 124.46 118.11 0)
 			(effects
@@
 			)
 		)
-		(property "Description" "Power symbol creates a global label with name \"Earth\""
+		(property "Description" "Power symbol creates a global label with name \"GND\""
 			(at 124.46 113.03 0)
 			(effects

Commit message: Done a lot of work, connected all traces
Connections:
- net OUTN: now also FB3.1, U3.10 (OUTN)
- net OUTP: now also FB2.1, U3.9 (OUTP)
Changed lines of the file:
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@@
+		)
+	)
+	(label "OUTN"
+		(at 156.21 104.14 0)
+		(effects
+			(font
+				(size 1.27 1.27)
+			)
+			(justify left bottom)
+		)
+	)
+	(label "OUTP"
+		(at 156.21 96.52 0)
+		(effects
+			(font
+				(size 1.27 1.27)
+			)
+			(justify left bottom)
 		)
 	)
