File: nRF_beacon/AUDIO.kicad_sch (KiCad schematic)
At the start: 8 parts, among them U3 MAX98357A

Commit message: Adjustments to GPIO connector. Added testpads. Polygon pour by antenna for correct impedance matching
Parts:
- added TP10: VDD_AUDIO, TestPoint:TestPoint_Pad_D1.0mm, symbol Connector:TestPoint
Connections:
- net VDD_AUDIO: now also TP10.1
Changed lines of the file:
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@@
+	)
+	(symbol
+		(lib_id "Connector:TestPoint")
+		(at 172.72 78.74 270)
+		(unit 1)
+		(exclude_from_sim no)
+		(in_bom yes)
+		(on_board yes)
+		(dnp no)
+		(property "Reference" "TP10"
+			(at 173.99 76.962 90)
+			(effects
+				(font
+					(size 1.27 1.27)
+				)
+				(justify left)
+			)
+		)
+		(property "Value" "VDD_AUDIO"
+			(at 173.99 80.772 90)
+			(effects
+				(font
+					(size 1.27 1.27)
+				)
+				(justify left)
+			)
+		)
+		(property "Footprint" "TestPoint:TestPoint_Pad_D1.0mm"
+			(at 172.72 83.82 0)
+			(effects
+				(font
+					(size 1.27 1.27)
+				)
+				(hide yes)
+			)
+		)
+		(property "Datasheet" "~"
+			(at 172.72 83.82 0)
+			(effects
+				(font
+					(size 1.27 1.27)
+				)
+				(hide yes)
+			)
+		)
+		(property "Description" "test point"
+			(at 172.72 78.74 0)
+			(effects
+				(font
+					(size 1.27 1.27)
+				)
+				(hide yes)
+			)
+		)
+		(pin "1"
+		)
+		(instances
+			(project ""
+				(path "/1290e5f5-b91f-4d6e-b440-6b78e8fdc212/437e71df-bd9b-467f-b101-39f98a623051"
+					(reference "TP10")
+					(unit 1)
+				)
+			)
+		)
 	)
 	(symbol

Commit message: Added stitching vias and completed DRC tests
Other:
- company: (none) -> Mathias Ekse
- title: (none) -> I2S Audio Output
Changed lines of the file:
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@@
 	(generator_version "9.0")
 	(paper "A4")
+	(title_block
+		(title "I2S Audio Output")
+		(date "2026-03-07")
+		(rev "A")
+		(company "Mathias Ekse")
+		(comment 1 "Audio Interface")
+		(comment 2 "MAX98357A DAC")
+		(comment 3 "I2S Audio")
+		(comment 4 "Speaker Output")
+	)
+	(rectangle
+		(start 90.17 60.325)
+		(end 219.71 128.905)
+		(stroke
+			(width 0)
+			(type default)
+		)
+		(fill
+			(type none)
+		)
+	)
 	(text "Gain:\nVDD ~ 100kOhm - 3 dB\nVDD - 6 dB\nUnconnected - 9 dB\nGND - 12 dB (Foreløpig valg)\nGnd ~ 100kOhm - 15 dB"
 		(exclude_from_sim no)
