File: nRF_beacon/MCU.kicad_sch (KiCad schematic)
At the start: 22 parts, among them U1 nRF54L15-QFAA, X1 32MHz, X2 32.768 kHz

Commit message: Done a lot of work, connected all traces
Connections:
- net SCL: now also U1.39 (P1.11/AIN4/CK); no longer U1.40 (P1.12/AIN5/CK)
- net SDA: now also U1.40 (P1.12/AIN5/CK); no longer U1.39 (P1.11/AIN4/CK)
Changed lines of the file:
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@@
 		)
 	)
-	(hierarchical_label "SDA"
+	(hierarchical_label "SCL"
 		(shape input)
 		(at 229.87 60.96 0)
@@
 		)
 	)
-	(hierarchical_label "SCL"
+	(hierarchical_label "SDA"
 		(shape input)
 		(at 229.87 63.5 0)

Commit message: Continued fixing DRC errors. Increased trace width on several lines
Parts:
- U1: footprint Ekse:QFN48_6X6_NOR -> Ekse:QFN-48_EP_6x6_Pitch0.4mm
Changed lines of the file:
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@@
 			)
 		)
-		(property "Footprint" "Ekse:QFN48_6X6_NOR"
+		(property "Footprint" "Ekse:QFN-48_EP_6x6_Pitch0.4mm"
 			(at 55.88 86.36 0)
 			(effects
@@
 			)
 		)
-		(property "Footprint" "Ekse:QFN48_6X6_NOR"
+		(property "Footprint" "Ekse:QFN-48_EP_6x6_Pitch0.4mm"
 			(at 195.58 116.84 0)
 			(effects
@@
 			)
 		)
-		(property "Footprint" "Ekse:QFN48_6X6_NOR"
+		(property "Footprint" "Ekse:QFN-48_EP_6x6_Pitch0.4mm"
 			(at 196.85 142.24 0)
 			(effects
@@
 			)
 		)
-		(property "Footprint" "Ekse:QFN48_6X6_NOR"
+		(property "Footprint" "Ekse:QFN-48_EP_6x6_Pitch0.4mm"
 			(at 223.52 71.12 0)
 			(effects

Commit message: Adjustments to GPIO connector. Added testpads. Polygon pour by antenna for correct impedance matching
Parts:
- added TP1: VDD_nRF, TestPoint:TestPoint_Pad_D1.0mm, symbol Connector:TestPoint
- added TP3: DECA, TestPoint:TestPoint_Pad_D1.0mm, symbol Connector:TestPoint
Connections:
- net VDD_nRF: now also TP1.1
- net at C1.1, C3.1, C5.1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: now also TP3.1
Changed lines of the file:
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@@
 	)
 	(junction
+		(at 41.91 38.1)
+		(diameter 0)
+		(color 0 0 0 0)
+	)
+	(junction
 		(at 104.14 78.74)
 		(diameter 0)
@@
 	(wire
 		(pts
-			(xy 31.75 38.1) (xy 50.8 38.1)
+			(xy 31.75 38.1) (xy 41.91 38.1)
 		)
 		(stroke
@@
 	(wire
 		(pts
+			(xy 41.91 38.1) (xy 50.8 38.1)
+		)
+		(stroke
+			(width 0)
+			(type default)
+		)
+	)
+	(wire
+		(pts
 			(xy 21.59 38.1) (xy 31.75 38.1)
 		)
@@
 	)
 	(symbol
+		(lib_id "Connector:TestPoint")
+		(at 19.05 72.39 90)
+		(unit 1)
+		(exclude_from_sim no)
+		(in_bom yes)
+		(on_board yes)
+		(dnp no)
+		(property "Reference" "TP3"
+			(at 15.748 70.612 90)
+			(effects
+				(font
+					(size 1.27 1.27)
+				)
+			)
+		)
+		(property "Value" "DECA"
+			(at 15.748 74.422 90)
+			(effects
+				(font
+					(size 1.27 1.27)
+				)
+			)
+		)
+		(property "Footprint" "TestPoint:TestPoint_Pad_D1.0mm"
+			(at 19.05 67.31 0)
+			(effects
+				(font
+					(size 1.27 1.27)
+				)
+				(hide yes)
+			)
+		)
+		(property "Datasheet" "~"
+			(at 19.05 67.31 0)
+			(effects
+				(font
+					(size 1.27 1.27)
+				)
+				(hide yes)
+			)
+		)
+		(property "Description" "test point"
+			(at 19.05 72.39 0)
+			(effects
+				(font
+					(size 1.27 1.27)
+				)
+				(hide yes)
+			)
+		)
+		(pin "1"
+		)
+		(instances
+			(project ""
+				(path "/1290e5f5-b91f-4d6e-b440-6b78e8fdc212/eb04787d-40f4-45c6-8e79-38c58cd136de"
+					(reference "TP3")
+					(unit 1)
+				)
+			)
+		)
+	)
+	(symbol
 		(lib_id "power:Earth")
 		(at 115.57 45.72 0)
@@
 					(unit 1)
 				)
+			)
+		)
+	)
+	(symbol
+		(lib_id "Connector:TestPoint")
+		(at 41.91 38.1 0)
+		(unit 1)
+		(exclude_from_sim no)
+		(in_bom yes)
+		(on_board yes)
+		(dnp no)
+		(fields_autoplaced yes)
+		(property "Reference" "TP1"
+			(at 44.45 33.5279 0)
+			(effects
+				(font
+					(size 1.27 1.27)
+				)
+				(justify left)
+			)
+		)
+		(property "Value" "VDD_nRF"
+			(at 44.45 36.0679 0)
+			(effects
+				(font
+					(size 1.27 1.27)
+				)
+				(justify left)
+			)
+		)
+		(property "Footprint" "TestPoint:TestPoint_Pad_D1.0mm"
+			(at 46.99 38.1 0)
+			(effects
+				(font
+					(size 1.27 1.27)
+				)
+				(hide yes)
+			)
+		)
+		(property "Datasheet" "~"
+			(at 46.99 38.1 0)
+			(effects
+				(font
+					(size 1.27 1.27)
+				)
+				(hide yes)
+			)
+		)
+		(property "Description" "test point"
+			(at 41.91 38.1 0)
+			(effects
+				(font
+					(size 1.27 1.27)
+				)
+				(hide yes)
+			)
+		)
+		(pin "1"
+		)
+		(instances
+			(project ""
+				(path "/1290e5f5-b91f-4d6e-b440-6b78e8fdc212/eb04787d-40f4-45c6-8e79-38c58cd136de"
+					(reference "TP1")
+					(unit 1)
+				)

Commit message: Added stitching vias and completed DRC tests
Other:
- note added: "P0 - NOT USED"
- note added: "P1 - Peripherals"
- note added: "P2 - NOT USED"
- note added: "nRF54L15 TYPICAL APPLICATION"
- note removed: "P1"
- note removed: "Vurder KGM15BR72A104KT"
- note removed: "nRF54L15 GENERAL APPLICATION"
- company: (none) -> Mathias Ekse
- title: (none) -> nRF54L15 MCU and RF Section
- moved on the sheet: C1, C10, C11, C12, C13, C2, C3, C4, C5, C6, C7, C8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

Commit message: Completed layout for Revision A (Prototype). Created gerber files
Parts:
- added H1, H2: MountingHole, MountingHole:MountingHole_3.2mm_M3_Pad_Via, symbol Mechanical:MountingHole
- added H3, H4: MountingHole, MountingHole:MountingHole_3.2mm_M3, symbol Mechanical:MountingHole
- added TP9: GND, TestPoint:TestPoint_Pad_D1.0mm, symbol Connector:TestPoint
Connections:
- net GND: now also TP9.1
Other:
- note added: "EXTRA"
